File: Garaż.kicad_pcb (KiCad board)
At the start: 2 copper layers, 90 x 100 mm, 32 parts, among them J1 AC L/N, J2 Gate, K1 Relay_SPST-NC, K2 Relay_SPST-NC, Q1 2N5551, Q2 2N5551, SW1 Button, SW2 Radio, U1 LM2940T-5.0/NOPB, U2 ACS712xLCTR-05B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

Commit message: Working project
Parts:
- C4: value 100nF -> 22uF
- K1, K2: value Relay_SPST-NC -> Relay_SPST-NO
- R3, R4: value 47k -> 68k
- moved J2 7.88 mm to (69.2, 54.6)
- moved J1 6.92 mm to (85.7, 54.7)
- moved Q1 2.48 mm to (111.8, 91.4), turned to 180 degrees
- moved Q2 2.48 mm to (118.7, 91.4), turned to 180 degrees
Connections:
- Q1 pad 1: Net-(Q1-C) -> GND
- Q1 pad 3: GND -> Net-(Q1-C)
- Q2 pad 1: Net-(Q2-C) -> GND
- Q2 pad 3: GND -> Net-(Q2-C)
Routing:
- net AC/N: track 169.0 -> 147.3 mm
- net AC/G2: track 32.4 -> 24.4 mm
- net AC/L: track 115.4 -> 108.3 mm
- net AC/G1: track 23.9 -> 20.7 mm
Other:
- outline, holes or cut-outs redrawn
