File: Garaż.kicad_sch (KiCad schematic)
At the start: 32 parts, among them J1 AC L/N, J2 Gate, K1 Relay_SPST-NC, K2 Relay_SPST-NC, Q1 2N5551, Q2 2N5551, SW1 Button, SW2 Radio, U1 LM2940T-5.0/NOPB, U2 ACS712xLCTR-05B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

Commit message: Add simulation
Parts:
- C4: value 100nF -> 22uF
- R1, R2: value 10k -> 6k8
- R3, R4: value 47k -> 51k
Changed lines of the file:
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@@
 			)
 		)
-		(property "Value" "10k"
+		(property "Value" "6k8"
 			(at 146.05 125.73 90)
 			(effects
@@
 			)
 		)
-		(property "Value" "10k"
+		(property "Value" "6k8"
 			(at 146.05 148.59 90)
 			(effects
@@
 			)
 		)
-		(property "Value" "47k"
+		(property "Value" "51k"
 			(at 154.94 133.3501 0)
 			(effects
@@
 			)
 		)
-		(property "Value" "100nF"
+		(property "Value" "22uF"
 			(at 212.09 142.6209 0)
 			(effects
@@
 			)
 		)
-		(property "Value" "47k"
+		(property "Value" "51k"
 			(at 168.91 148.59 90)
 			(effects

Commit message: Working project
Parts:
- removed K1, K2: Relay_SPST-NC, Relay_THT:Relay_SPST_Panasonic_JW1_FormA, symbol Relay:Relay_SPST-NC
- added K1, K2: Relay_SPST-NO, Relay_THT:Relay_SPST_Panasonic_JW1_FormA, symbol Relay:Relay_SPST-NO
- R1, R2: value 6k8 -> 10k
- R3, R4: value 51k -> 68k
Connections:
- net +12V: now also K1.8, K2.8
- net AC/G1: now also K1.6
- net AC/G2: now also K2.6
- net AC/L: now also K1.4, K2.4
- net GND: now also Q1.1 (E), Q2.1 (E); no longer Q1.3 (E), Q2.3 (E)
- new net: K1.1, Q1.3 (C)
- new net: K2.1, Q2.3 (C)
Changed lines of the file:
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@@
 	(wire
 		(pts
-			(xy 182.88 72.39) (xy 182.88 85.09)
-		)
-		(stroke
-			(width 0)
-			(type default)
-		)
-	)
-	(wire
-		(pts
 			(xy 172.72 152.4) (xy 184.15 152.4)
 		)
@@
 	(wire
 		(pts
-			(xy 151.13 72.39) (xy 151.13 100.33)
-		)
-		(stroke
-			(width 0)
-			(type default)
-		)
-	)
-	(wire
-		(pts
 			(xy 184.15 132.08) (xy 186.69 132.08)
 		)
@@
 	(wire
 		(pts
+			(xy 151.13 74.93) (xy 151.13 100.33)
+		)
+		(stroke
+			(width 0)
+			(type default)
+		)
+	)
+	(wire
+		(pts
 			(xy 196.85 132.08) (xy 196.85 138.43)
 		)
@@
 	(wire
 		(pts
+			(xy 182.88 74.93) (xy 182.88 85.09)
+		)
+		(stroke
+			(width 0)
+			(type default)
+		)
+	)
+	(wire
+		(pts
 			(xy 30.48 49.53) (xy 153.67 49.53)
 		)
@@
 	)
 	(symbol
+		(lib_id "Relay:Relay_SPST-NO")
+		(at 143.51 69.85 270)
+		(mirror x)
+		(unit 1)
+		(exclude_from_sim no)
+		(in_bom yes)
+		(on_board yes)
+		(dnp no)
+		(property "Reference" "K1"
+			(at 143.51 54.61 90)
+			(effects
+				(font
+					(size 1.27 1.27)
+				)
+			)
+		)
+		(property "Value" "Relay_SPST-NO"
+			(at 143.51 57.15 90)
+			(effects
+				(font
+					(size 1.27 1.27)
+				)
+			)
+		)
+		(property "Footprint" "Relay_THT:Relay_SPST_Panasonic_JW1_FormA"
+			(at 142.24 58.42 0)
+			(effects
+				(font
+					(size 1.27 1.27)
+				)
+				(justify left)
+				(hide yes)
+			)
+		)
+		(property "Datasheet" "~"
+			(at 143.51 69.85 0)
+			(effects
+				(font
+					(size 1.27 1.27)
+				)
+				(hide yes)
+			)
+		)
+		(property "Description" "Relay SPST, normally open, EN50005"
+			(at 143.51 69.85 0)
+			(effects
+				(font
+					(size 1.27 1.27)
+				)
+				(hide yes)
+			)
+		)
+		(pin "4"
+		)
+		(pin "1"
+		)
+		(pin "8"
+		)
+		(pin "6"
+		)
+		(instances
+			(project ""
+				(path "/8f3f2cb0-c7c7-4116-9663-55f4dfa53e17"
+					(reference "K1")
+					(unit 1)
+				)
+			)
+		)
+	)
+	(symbol
 		(lib_id "Device:D")
 		(at 66.04 96.52 90)
@@
 			)
 		)
-		(property "Value" "6k8"
+		(property "Value" "10k"
 			(at 146.05 125.73 90)
 			(effects
@@
 			)
 		)
-		(property "Value" "6k8"
+		(property "Value" "10k"
 			(at 146.05 148.59 90)
 			(effects
@@
 	)
 	(symbol
-		(lib_id "Relay:Relay_SPST-NC")
-		(at 175.26 67.31 90)
-		(unit 1)
-		(exclude_from_sim no)
-		(in_bom yes)
-		(on_board yes)
-		(dnp no)
-		(property "Reference" "K2"
-			(at 175.26 52.07 90)
-			(effects
-				(font
-					(size 1.27 1.27)
-				)
-			)
-		)
-		(property "Value" "Relay_SPST-NC"
-			(at 175.26 54.61 90)
-			(effects
-				(font
-					(size 1.27 1.27)
-				)
-			)
-		)
-		(property "Footprint" "Relay_THT:Relay_SPST_Panasonic_JW1_FormA"
-			(at 176.53 55.88 0)
-			(effects
-				(font
-					(size 1.27 1.27)
-				)
-				(justify left)
-				(hide yes)
-			)
-		)
-		(property "Datasheet" "~"
-			(at 175.26 67.31 0)
-			(effects
-				(font
-					(size 1.27 1.27)
-				)
-				(hide yes)
-			)
-		)
-		(property "Description" "Relay SPST, normally closed, EN50005"
-			(at 175.26 67.31 0)
-			(effects
-				(font
-					(size 1.27 1.27)
-				)
-				(hide yes)
-			)
-		)
-		(pin "6"
-		)
-		(pin "4"
-		)
-		(pin "8"
-		)
-		(pin "1"
-		)
-		(instances
-			(project "Garaż"
-				(path "/8f3f2cb0-c7c7-4116-9663-55f4dfa53e17"
-					(reference "K2")
-					(unit 1)
-				)
-			)
-		)
-	)
-	(symbol
 		(lib_id "Mechanical:MountingHole")
 		(at 213.36 44.45 0)
@@
 			)
 		)
-		(property "Value" "51k"
+		(property "Value" "68k"
 			(at 154.94 133.3501 0)
 			(effects
@@
 	)
 	(symbol
+		(lib_name "NPN_1")
 		(lib_id "Simulation_SPICE:NPN")
 		(at 153.67 105.41 0)
@@
 			)
 		)
-		(property "Value" "51k"
+		(property "Value" "68k"
 			(at 168.91 148.59 90)
 			(effects
@@
 	)
 	(symbol
-		(lib_id "Relay:Relay_SPST-NC")
-		(at 143.51 67.31 90)
-		(unit 1)
-		(exclude_from_sim no)
-		(in_bom yes)
-		(on_board yes)
-		(dnp no)
-		(property "Reference" "K1"
-			(at 143.51 52.07 90)
-			(effects
-				(font
-					(size 1.27 1.27)
-				)
-			)
-		)
-		(property "Value" "Relay_SPST-NC"
-			(at 143.51 54.61 90)
-			(effects
-				(font
-					(size 1.27 1.27)
-				)
-			)
-		)
-		(property "Footprint" "Relay_THT:Relay_SPST_Panasonic_JW1_FormA"
-			(at 144.78 55.88 0)
-			(effects
-				(font
-					(size 1.27 1.27)
-				)
-				(justify left)
-				(hide yes)
-			)
-		)
-		(property "Datasheet" "~"
-			(at 143.51 67.31 0)
-			(effects
-				(font
-					(size 1.27 1.27)
-				)
-				(hide yes)
-			)
-		)
-		(property "Description" "Relay SPST, normally closed, EN50005"
-			(at 143.51 67.31 0)
-			(effects
-				(font
-					(size 1.27 1.27)
-				)
-				(hide yes)
-			)
-		)
-		(pin "6"
-		)
-		(pin "4"
-		)
-		(pin "8"
-		)
-		(pin "1"
-		)
-		(instances
-			(project ""
-				(path "/8f3f2cb0-c7c7-4116-9663-55f4dfa53e17"
-					(reference "K1")
-					(unit 1)
-				)
-			)
-		)
-	)
-	(symbol
 		(lib_id "power:+5V")
 		(at 238.76 105.41 270)
@@
 	)
 	(symbol
+		(lib_id "Relay:Relay_SPST-NO")
+		(at 175.26 69.85 270)
+		(mirror x)
+		(unit 1)
+		(exclude_from_sim no)
+		(in_bom yes)
+		(on_board yes)
+		(dnp no)
+		(property "Reference" "K2"
+			(at 175.26 54.61 90)
+			(effects
+				(font
+					(size 1.27 1.27)
+				)
+			)
+		)
+		(property "Value" "Relay_SPST-NO"
+			(at 175.26 57.15 90)
+			(effects
+				(font
+					(size 1.27 1.27)
+				)
+			)
+		)
+		(property "Footprint" "Relay_THT:Relay_SPST_Panasonic_JW1_FormA"
+			(at 173.99 58.42 0)
+			(effects
+				(font
+					(size 1.27 1.27)
+				)
+				(justify left)
+				(hide yes)
+			)
+		)
+		(property "Datasheet" "~"
+			(at 175.26 69.85 0)
+			(effects
+				(font
+					(size 1.27 1.27)
+				)
+				(hide yes)
+			)
+		)
+		(property "Description" "Relay SPST, normally open, EN50005"
+			(at 175.26 69.85 0)
+			(effects
+				(font
+					(size 1.27 1.27)
+				)
+				(hide yes)
+			)
+		)
+		(pin "4"
+		)
+		(pin "1"
+		)
+		(pin "8"
+		)
+		(pin "6"
+		)
+		(instances
+			(project "Garaż"
+				(path "/8f3f2cb0-c7c7-4116-9663-55f4dfa53e17"
+					(reference "K2")
+					(unit 1)
+				)
+			)
+		)
+	)
+	(symbol
 		(lib_id "power:GND")
 		(at 54.61 113.03 0)
@@
 	(symbol
 		(lib_id "power:+6V")
-		(at 167.64 72.39 90)
+		(at 167.64 74.93 90)
 		(unit 1)
 		(exclude_from_sim no)
@@
 		(dnp no)
 		(property "Reference" "#PWR011"
-			(at 171.45 72.39 0)
+			(at 171.45 74.93 0)
 			(effects
 				(font
@@
 		)
 		(property "Value" "+12V"
-			(at 163.83 72.3899 90)
+			(at 163.83 74.9299 90)
 			(effects
 				(font
@@
 		)
 		(property "Footprint" ""
-			(at 167.64 72.39 0)
+			(at 167.64 74.93 0)
 			(effects
 				(font
@@
 		)
 		(property "Datasheet" ""
-			(at 167.64 72.39 0)
+			(at 167.64 74.93 0)
 			(effects
 				(font
@@
 		)
 		(property "Description" "Power symbol creates a global label with name \"+6V\""
-			(at 167.64 72.39 0)
+			(at 167.64 74.93 0)
 			(effects
 				(font
@@
 	(symbol
 		(lib_id "power:+6V")
-		(at 135.89 72.39 90)
+		(at 135.89 74.93 90)
 		(unit 1)
 		(exclude_from_sim no)
@@
 		(dnp no)
 		(property "Reference" "#PWR06"
-			(at 139.7 72.39 0)
+			(at 139.7 74.93 0)
 			(effects
 				(font
@@
 		)
 		(property "Value" "+12V"
-			(at 132.08 72.3899 90)
+			(at 132.08 74.9299 90)
 			(effects
 				(font
@@
 		)
 		(property "Footprint" ""
-			(at 135.89 72.39 0)
+			(at 135.89 74.93 0)
 			(effects
 				(font
@@
 		)
 		(property "Datasheet" ""
-			(at 135.89 72.39 0)
+			(at 135.89 74.93 0)
 			(effects
 				(font
@@
 		)
 		(property "Description" "Power symbol creates a global label with name \"+6V\""
-			(at 135.89 72.39 0)
+			(at 135.89 74.93 0)
 			(effects
 				(font
