File: symulacja.kicad_sch (KiCad schematic)
At the start: 12 parts, among them U1 ${SIM.PARAMS}

Commit message: Working project
Parts:
- R1, R2: value 6k8 -> 10k
- R3, R4: value 51k -> 68k
Changed lines of the file:
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@@
+			)
+		)
+		(property "Sim.Params" "GAIN=140k"
+			(at 147.32 92.71 0)
+			(effects
+				(font
+					(size 1.27 1.27)
+				)
+				(hide yes)
 			)
 		)
@@
 			)
 		)
-		(property "Value" "6k8"
+		(property "Value" "10k"
 			(at 123.19 86.36 90)
 			(effects
@@
 			)
 		)
-		(property "Value" "6k8"
+		(property "Value" "10k"
 			(at 129.54 109.22 90)
 			(effects
@@
 			)
 		)
-		(property "Value" "51k"
+		(property "Value" "68k"
 			(at 133.35 96.5199 0)
 			(effects
@@
 			)
 		)
-		(property "Value" "51k"
+		(property "Value" "68k"
 			(at 146.05 109.22 90)
 			(effects
